Commit message: phase 4: dynamics engine (rnea, crba, forward dynamics, simulator)
caliper-spatial: SpatialInertia (6x6, [v;w] order) with covariant transform
(the fixed-link inertia fold) + KE-invariance test.
caliper-model: parse urdf <inertial> into per-movable-link spatial inertia,
folding fixed-welded descendants onto their movable parent along the same
compile() DFS; has_inertia gate; missing-inertial = mass<=0 treated absent.
caliper-dynamics: body-frame RNEA (inverse dynamics + gravity), CRBA (mass
matrix), forward dynamics (crba + rnea-bias + cholesky), and a semi-implicit/
rk4 Simulator (gravity, viscous damping, applied torque, finiteness guards).
fixtures: showcase6 <inertial> added (kinematics unchanged), dyn_pendulum2
(analytic 2R), dyn_welded (fixed-fold cross-val vs pinocchio).
self-validated: crba column == rnea unit-accel, fd round-trip 1e-9, rk4
passive-swing energy <3e-3, spd/symmetry. 59 rust tests, clippy -D, fmt.

File: oracle/fixtures/robots/showcase6.urdf (robot description, URDF)
Before this commit: robot showcase6, 7 links, 6 joints
Links:
- link base: mass None -> 2.0
- link flange: mass None -> 0.3
- link forearm: mass None -> 0.9
- link shoulder: mass None -> 1.6
- link upper_arm: mass None -> 1.2
- link wrist1: mass None -> 0.5
- link wrist2: mass None -> 0.4
